File: HB-UNI-Sen-WEA/HB-UNI-Sen-WEA.kicad_pcb (KiCad board)
At the start: 2 copper layers, 66 x 55.9 mm, 23 parts, among them J1 RAIN, J10 BATT, J2 PROG, J3 WIND_DIR, J4 I2C_1, J5 LIGHTNING, J6 ANEM, J7 RAIN_Q, J8 I2C_2, J9 I2C_3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

Commit message: new pcb routing
Parts:
- MH1, MH2: value MountingHole_2.2mm_M2_Pad_Via -> MountingHole_2.2mm_M2; footprint MountingHole:MountingHole_2.2mm_M2_Pad_Via -> MountingHole:MountingHole_2.2mm_M2
- moved MH2 37.4 mm to (130.8, 116.8)
Routing:
- net GND: track 211.9 -> 4.17 mm, vias 0 -> 6
- net /A3: track 108.1 -> 44.5 mm
- net +5V: track 122.7 -> 72.6 mm
- net /D6: track 61.2 -> 94.9 mm, vias 1 -> 0
- net /SCL: track 94.3 -> 83.2 mm
- net /D5: track 62.9 -> 72.4 mm
- net /SDA: track 91.5 -> 100.5 mm, vias 0 -> 1
- net /VCC: track 120.3 -> 114.0 mm
- net /D3: track 38.9 -> 34.0 mm
- net /MISO: track 52.1 -> 47.9 mm
- net /D2: track 39.2 -> 35.5 mm
- net /SS: track 20.4 -> 22.5 mm
- net /D7: track 29.6 -> 27.9 mm
- net /MOSI: track 55.8 -> 54.7 mm, vias 1 -> 0
- net /D8: track 36.7 -> 35.7 mm
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Other:
- outline, holes or cut-outs redrawn
